File: Hardware/v2/f91_kepler_v2.kicad_pcb (KiCad board)
At the start: 2 copper layers, 25 x 27 mm, 89 parts, among them J1 LS013B7DH03 FPC, Q1 FS8205A, SW1 BTN1/BSL, SW2 BTN2, SW3 BTN3, U1 CC2652R7RGZ, U2 BQ51050B, U3 DW01A, U4 XC6206P302MR, U5 LIS2DW12, U6 DRV2605L, U7 ST25DV04K, Y1 48MHz FA-128, Y2 32.768kHz FC-135

Commit message: fix(hw/v2): close PCB<->schematic parity debt (123 -> 1)
Board was generated with blank footprint library nicknames and a few
metadata gaps, producing 123 schematic-parity mismatches that would fight
"update PCB from schematic". Closed almost all:

- fix_fpids.py: set each board footprint FPID nickname from the schematic
  (item names already matched -> no geometry change). Clears 105 name
  mismatches.
- fix_tp_bom.py: TP1-16 symbols in_bom/in_pos_files yes -> no. Test points
  (pogo pads + taps) are not orderable BOM parts; the footprints already
  excluded them. Clears 16 attribute mismatches.
- fix_unconnected_nets.py: assign the schematic's single-pad
  "unconnected-(...)" nets (spare U1/U2/U3/U5/U7 pins) to the matching
  netless board pads. Clears 17 net_conflicts.

Remaining (all benign, documented):
- parity 1: U7 ST25DV symbol pin 9 = "NC" (hidden); SO8 footprint correctly
  has no pad 9. KiCad flags NC pins without pads as warnings.
- ERC 2: U4 lib_symbol_mismatch (stale embedded copy vs Regulator_Linear;
  fix via Eeschema "Update Symbols from Library"); U5 pin_to_pin (SDO/SA0
  tied to GND for I2C address select — intentional, ERC false positive).

DRC fab-blocking still 0. Schematic migrated f91gen -> eeschema format.
Parts:
- AE1: footprint ANT_2450AT18A100 -> f91_footprints:ANT_2450AT18A100
- BT1: footprint BatteryPads -> f91_footprints:BatteryPads
- C10, C11, C12, C13, C14, C15, C18, C2, C21, C22, C23, C24, C25, C26, C27, C28, C29, C3, C30, C31, C32, C33, C34, C35, C36, C37, C38, C39, C4, C40, C6, C8, C9: footprint C_0402_1005Metric -> Capacitor_SMD:C_0402_1005Metric
- C16, C17, C19, C20, C5, C7: footprint C_0603_1608Metric -> Capacitor_SMD:C_0603_1608Metric
- FB1: footprint L_0603_1608Metric -> Inductor_SMD:L_0603_1608Metric
- FL1: footprint Murata_LFB18_1608 -> f91_footprints:Murata_LFB18_1608
- J1: footprint Hirose_FH12-10S-0.5SH_1x10-1MP_P0.50mm_Horizontal -> Connector_FFC-FPC:Hirose_FH12-10S-0.5SH_1x10-1MP_P0.50mm_Horizontal
- L2: footprint L_0805_2012Metric -> Inductor_SMD:L_0805_2012Metric
- Q1: footprint TSSOP-8_3x3mm_P0.65mm -> Package_SO:TSSOP-8_3x3mm_P0.65mm
- R1, R10, R11, R12, R13, R14, R2, R3, R4, R5, R6, R7, R8, R9, W1: footprint R_0402_1005Metric -> Resistor_SMD:R_0402_1005Metric
- SW1, SW2, SW3: footprint SW_Push_1P1T_NO_CK_KMR2 -> Button_Switch_SMD:SW_Push_1P1T_NO_CK_KMR2
- TP1, TP10, TP11, TP12, TP13, TP14, TP15, TP16, TP2, TP3, TP4, TP5, TP6, TP7, TP8, TP9: footprint TestPoint_Pad_1.5x1.5mm -> TestPoint:TestPoint_Pad_1.5x1.5mm
- U1: footprint QFN-48-1EP_7x7mm_P0.5mm_EP5.15x5.15mm -> Package_DFN_QFN:QFN-48-1EP_7x7mm_P0.5mm_EP5.15x5.15mm
- U2: footprint VQFN-20-1EP_4.5x3.5mm_P0.5mm -> f91_footprints:VQFN-20-1EP_4.5x3.5mm_P0.5mm
- U3: footprint SOT-23-6 -> Package_TO_SOT_SMD:SOT-23-6
- U4: footprint SOT-23 -> Package_TO_SOT_SMD:SOT-23
- U5: footprint LGA-12_2x2mm_P0.5mm -> Package_LGA:LGA-12_2x2mm_P0.5mm
- U6: footprint VSSOP-10_3x3mm_P0.5mm -> f91_footprints:VSSOP-10_3x3mm_P0.5mm
- U7: footprint SOIC-8_3.9x4.9mm_P1.27mm -> Package_SO:SOIC-8_3.9x4.9mm_P1.27mm
- Y1: footprint Crystal_SMD_3215-4Pin_3.2x1.5mm -> f91_footprints:Crystal_SMD_3215-4Pin_3.2x1.5mm
- Y2: footprint Crystal_SMD_3215-2Pin_3.2x1.5mm -> Crystal:Crystal_SMD_3215-2Pin_3.2x1.5mm
Connections:
- U1 pad 26: (no net) -> unconnected-(U1-DIO_16-Pad26)
- U1 pad 27: (no net) -> unconnected-(U1-DIO_17-Pad27)
- U1 pad 28: (no net) -> unconnected-(U1-DIO_18-Pad28)
- U1 pad 29: (no net) -> unconnected-(U1-DIO_19-Pad29)
- U1 pad 30: (no net) -> unconnected-(U1-DIO_20-Pad30)
- U1 pad 36: (no net) -> unconnected-(U1-DIO_23-Pad36)
- U1 pad 40: (no net) -> unconnected-(U1-DIO_27-Pad40)
- U1 pad 41: (no net) -> unconnected-(U1-DIO_28-Pad41)
- U1 pad 42: (no net) -> unconnected-(U1-DIO_29-Pad42)
- U1 pad 43: (no net) -> unconnected-(U1-DIO_30-Pad43)
- U1 pad 5: (no net) -> unconnected-(U1-DIO_0-Pad5)
- U1 pad 6: (no net) -> unconnected-(U1-DIO_1-Pad6)
- U1 pad 9: (no net) -> unconnected-(U1-DIO_4-Pad9)
- U2 pad 8: (no net) -> unconnected-(U2-~{AD-EN}-Pad8)
- U3 pad 4: (no net) -> unconnected-(U3-TD-Pad4)
- U5 pad 5: (no net) -> unconnected-(U5-NC-Pad5)
- U7 pad 1: (no net) -> unconnected-(U7-V_EH-Pad1)
